File: WS2812Controller.kicad_pcb (KiCad board)
At the start: 2 copper layers, 49.4 x 35.8 mm, 22 parts, among them J1 Conn_01x04_Male, J2 Conn_01x05_Male, J3 Conn_01x03, SW1 SW_Reset, SW2 SW_GPIO0, U1 AMS1117-3.3, U2 ESP-12F, U3 SN74AHCT125

Commit message: Updated working copy
Parts:
- removed G***: LOGO, halibs:Logo_20mm
- C1, C2: footprint Capacitor_SMD:C_0805_2012Metric_Pad1.15x1.40mm_HandSolder -> Capacitor_SMD:C_0805_2012Metric_Pad1.18x1.45mm_HandSolder
- F1: footprint halibs:Fuse-PTF75_Stelvio -> Custom Footprints CB:Fuse-PTF75_Stelvio
- R1, R2, R3, R4, R5, R6: footprint Resistor_SMD:R_0805_2012Metric_Pad1.15x1.40mm_HandSolder -> Resistor_SMD:R_0805_2012Metric_Pad1.20x1.40mm_HandSolder
- U3: footprint haus-automatisierung:SN74AHCT125D -> Custom Footprints CB:SN74AHCT125D
- moved U3 6.09 mm to (135.7, 75.0)
Routing:
- net GND: track 16.1 -> 3.08 mm, vias 2 -> 1
- net +5V: track 66.1 -> 63.0 mm, vias 1 -> 2
- net GPIO4: track 34.0 -> 32.4 mm
- net TX: track 8.17 -> 9.37 mm
- net +3V3: track 57.7 -> 58.8 mm
Other:
- board text removed: "haus-automatisierung.com"
